Commit message: Added controller packages and modified descriptions

File: inchworm_description/urdf/inchworm_description.urdf (robot description, URDF)
Before this commit: robot inchworm_description, 4 links, 3 joints
Links:
- added link link_4, mass 0.075697; collision mesh filename=package://inchworm_description/meshes/link_4.STL; visual mesh filename=package://inchworm_description/meshes/link_4.STL
- link base_link: mass 0.10777 -> None; geometry 
- link link_1: mass 0.12376 -> 0.10777
- link link_3: mass 0.075697 -> 0.12376
Joints:
- added joint fake_base_joint: type fixed, parent base_link, child link_1, origin xyz=0 0 0 rpy=0 0 0
- joint joint_1: child link_1 -> link_2; parent base_link -> link_1
- joint joint_2: child link_2 -> link_3; parent link_1 -> link_2
- joint joint_3: child link_3 -> link_4; parent link_2 -> link_3

Commit message: Added controllers, fixed scripts to spawn multiple models

File: inchworm_description/urdf/inchworm_description.urdf (robot description, URDF)
Before this commit: robot inchworm, 5 links, 4 joints
Joints:
- joint joint_1: limit lower=0 upper=0 effort=0 velocity=0 -> lower=0 upper=0 effort=30 velocity=0
- joint joint_2: limit lower=0 upper=0 effort=0 velocity=0 -> lower=0 upper=0 effort=30 velocity=0
- joint joint_3: limit lower=0 upper=0 effort=0 velocity=0 -> lower=0 upper=0 effort=30 velocity=0

Commit message: Working model of basic control

File: inchworm_description/urdf/inchworm_description.urdf (robot description, URDF)
Before this commit: robot inchworm, 5 links, 4 joints
Links:
- removed link base_link
- added link world
Joints:
- removed joint fake_base_joint
- added joint world_to_link_1: type fixed, parent world, child link_1, origin xyz=0 0 0 rpy=0 0 0

Commit message: Created a proper gravity comp + pd controller using rbdl

File: inchworm_description/urdf/inchworm_description.urdf (robot description, URDF)
Before this commit: robot inchworm, 5 links, 4 joints
Links:
- removed link world
Joints:
- removed joint world_to_link_1
- joint joint_1: axis 1 0 0 -> 1.0 0.0 0.0; limit lower=0 upper=0 effort=30 velocity=0 -> lower=0.0 upper=0.0 effort=30.0 velocity=0.0; origin xyz=0 -0.0002 0.10478 rpy=-3.1399 0 3.1416 -> xyz=0.0 -0.0002 0.10478 rpy=-3.1399 0.0 3.1416
- joint joint_2: axis -1 0 0 -> -1.0 0.0 0.0; limit lower=0 upper=0 effort=30 velocity=0 -> lower=0.0 upper=0.0 effort=30.0 velocity=0.0; origin xyz=-0.02165 -0.015204 -0.14832 rpy=0.00024788 0 0 -> xyz=-0.02165 -0.015204 -0.14832 rpy=0.00024788 0.0 0.0
- joint joint_3: axis -1 0 0 -> -1.0 0.0 0.0; limit lower=0 upper=0 effort=30 velocity=0 -> lower=0.0 upper=0.0 effort=30.0 velocity=0.0; origin xyz=0.0017 -0.00017056 -0.16329 rpy=-0.0019608 0 0 -> xyz=0.0017 -0.00017056 -0.16329 rpy=-0.0019608 0.0 0.0

Commit message: Modified controller

File: inchworm_description/urdf/inchworm_description.urdf (robot description, URDF)
Before this commit: robot inchworm, 4 links, 3 joints
Links:
- added link link_5, mass 1.0
Joints:
- added joint temp_joint: type fixed, parent link_4, child link_5, origin xyz=0.051962 0.02982944 -0.307162 rpy=0.0 0.0 0.0

File: inchworm_description/urdf/inchworm_description_unscaled.urdf (robot description, URDF)
Before this commit: robot inchworm, 4 links, 3 joints
Links:
- added link link_5, mass 1
Joints:
- added joint temp_joint: type fixed, parent link_4, child link_5, origin xyz=0.051962 0.02982944 -0.307162 rpy=0 0 0
